File: HeartRateSensor Eval Board - Si1141/HeartRateSensor Eval Board - Si1141.brd (EAGLE design)
At the start: 100 x 80 mm, 6 parts

Commit message: Finished board layout.
Parts:
- moved C2 43.0 mm to (13.2, 11.2), turned to 270 degrees
- moved LED1 38.9 mm to (14.7, 2.79), turned to 180 degrees
- moved R1 36.9 mm to (9.65, 12.2), turned to 180 degrees
- moved C1 34.9 mm to (6.10, 11.2), turned to 270 degrees
- moved SV1 31.3 mm to (2.79, 7.11), turned to 90 degrees
- moved U$1 27.4 mm to (10.9, 2.79), turned to 270 degrees
Connections:
- net GND: now also SV1.1
- net VCC: no longer SV1.1
Routing:
- net VCC: track 0.00 -> 32.2 mm
- net SDA: track 0.00 -> 13.0 mm
- net N$2: track 0.00 -> 12.7 mm
- net SCL: track 0.00 -> 11.0 mm
- net INT: track 0.00 -> 7.72 mm
- net N$1: track 0.00 -> 3.62 mm
- net GND: track 0.00 -> 2.05 mm, vias 0 -> 3
- added copper zone on layer 1, net GND
- added copper zone on layer 16, net GND
Other:
- board size 100 x 80 mm -> 15.5 x 13.7 mm
