File: HeartRateSensor Eval Board - Si1141/HeartRateSensor Eval Board - Si1141.sch (EAGLE design)
At the start: 6 parts

Commit message: Finished board layout.
Connections:
- net GND: now also SV1.1
- net VCC: no longer SV1.1
Changed lines of the file:
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@@
 <label x="-22.86" y="60.96" size="1.778" layer="95"/>
-</segment>
-<segment>
-<pinref part="SV1" gate="G$1" pin="1"/>
-<wire x1="-17.78" y1="50.8" x2="-25.4" y2="50.8" width="0.1524" layer="91"/>
-<label x="-22.86" y="50.8" size="1.778" layer="95"/>
 </segment>
 </net>
@@
 <wire x1="114.3" y1="63.5" x2="114.3" y2="60.96" width="0.1524" layer="91"/>
 </segment>
+<segment>
+<pinref part="SV1" gate="G$1" pin="1"/>
+<wire x1="-17.78" y1="50.8" x2="-25.4" y2="50.8" width="0.1524" layer="91"/>
+<label x="-22.86" y="50.8" size="1.778" layer="95"/>
+</segment>
 </net>
